File: testo2H.K/testo2H.K.kicad_sch (KiCad schematic)
At the start: 4 parts, among them Q1 NMOS, Q2 NMOS, Q3 NMOS, Q4 NMOS

Commit message: 更新
Connections:
- net at Q4.3 (S): now also Q2.3 (S)
- net at Q3.1 (D): now also Q1.1 (D)
Other:
- moved on the sheet: Q1, Q2, Q3, Q4
Changed lines of the file:
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@@
 (kicad_sch (version 20230121) (generator eeschema)
   (paper "A4")
-  (junction (at 116.332 73.66) (diameter 0) (color 0 0 0 0)
-  )
-  (wire (pts (xy 135.89 69.342) (xy 135.89 74.422))
+  (wire (pts (xy 132.08 67.31) (xy 132.08 72.39))
     (stroke (width 0) (type default))
   )
-  (wire (pts (xy 116.332 73.914) (xy 116.586 73.914))
+  (wire (pts (xy 111.76 82.55) (xy 132.08 82.55))
     (stroke (width 0) (type default))
   )
-  (wire (pts (xy 116.078 73.66) (xy 116.332 73.66))
+  (wire (pts (xy 111.76 57.15) (xy 132.08 57.15))
     (stroke (width 0) (type default))
   )
-  (wire (pts (xy 116.078 69.088) (xy 116.078 73.66))
+  (wire (pts (xy 111.76 67.31) (xy 111.76 72.39))
     (stroke (width 0) (type default))
   )
-  (wire (pts (xy 116.332 73.66) (xy 116.332 73.914))
-    (stroke (width 0) (type default))
-  )
-  (wire (pts (xy 116.586 73.914) (xy 116.586 73.66))
-    (stroke (width 0) (type default))
-  )
-  (symbol (lib_id "Simulation_SPICE:NMOS") (at 138.43 79.502 0) (mirror y) (unit 1)
+  (symbol (lib_id "Simulation_SPICE:NMOS") (at 134.62 77.47 0) (mirror y) (unit 1)
     (in_bom yes) (on_board yes) (dnp no) (fields_autoplaced)
-    (property "Reference" "Q4" (at 132.588 78.232 0)
+    (property "Reference" "Q4" (at 128.778 76.2 0)
       (effects (font (size 1.27 1.27)) (justify left))
     )
-    (property "Value" "NMOS" (at 132.588 80.772 0)
+    (property "Value" "NMOS" (at 128.778 78.74 0)
       (effects (font (size 1.27 1.27)) (justify left))
     )
-    (property "Footprint" "" (at 133.35 76.962 0)
+    (property "Footprint" "" (at 129.54 74.93 0)
       (effects (font (size 1.27 1.27)) hide)
     )
-    (property "Datasheet" "https://ngspice.sourceforge.io/docs/ngspice-manual.pdf" (at 138.43 92.202 0)
+    (property "Datasheet" "https://ngspice.sourceforge.io/docs/ngspice-manual.pdf" (at 134.62 90.17 0)
       (effects (font (size 1.27 1.27)) hide)
     )
-    (property "Sim.Device" "NMOS" (at 138.43 96.647 0)
+    (property "Sim.Device" "NMOS" (at 134.62 94.615 0)
       (effects (font (size 1.27 1.27)) hide)
     )
-    (property "Sim.Type" "VDMOS" (at 138.43 98.552 0)
+    (property "Sim.Type" "VDMOS" (at 134.62 96.52 0)
       (effects (font (size 1.27 1.27)) hide)
     )
-    (property "Sim.Pins" "1=D 2=G 3=S" (at 138.43 94.742 0)
+    (property "Sim.Pins" "1=D 2=G 3=S" (at 134.62 92.71 0)
       (effects (font (size 1.27 1.27)) hide)
     )
@@
     )
   )
-  (symbol (lib_id "Simulation_SPICE:NMOS") (at 138.43 64.262 0) (mirror y) (unit 1)
+  (symbol (lib_id "Simulation_SPICE:NMOS") (at 134.62 62.23 0) (mirror y) (unit 1)
     (in_bom yes) (on_board yes) (dnp no) (fields_autoplaced)
-    (property "Reference" "Q3" (at 132.588 62.992 0)
+    (property "Reference" "Q3" (at 128.778 60.96 0)
       (effects (font (size 1.27 1.27)) (justify left))
     )
-    (property "Value" "NMOS" (at 132.588 65.532 0)
+    (property "Value" "NMOS" (at 128.778 63.5 0)
       (effects (font (size 1.27 1.27)) (justify left))
     )
-    (property "Footprint" "" (at 133.35 61.722 0)
+    (property "Footprint" "" (at 129.54 59.69 0)
       (effects (font (size 1.27 1.27)) hide)
     )
-    (property "Datasheet" "https://ngspice.sourceforge.io/docs/ngspice-manual.pdf" (at 138.43 76.962 0)
+    (property "Datasheet" "https://ngspice.sourceforge.io/docs/ngspice-manual.pdf" (at 134.62 74.93 0)
       (effects (font (size 1.27 1.27)) hide)
     )
-    (property "Sim.Device" "NMOS" (at 138.43 81.407 0)
+    (property "Sim.Device" "NMOS" (at 134.62 79.375 0)
       (effects (font (size 1.27 1.27)) hide)
     )
-    (property "Sim.Type" "VDMOS" (at 138.43 83.312 0)
+    (property "Sim.Type" "VDMOS" (at 134.62 81.28 0)
       (effects (font (size 1.27 1.27)) hide)
     )
-    (property "Sim.Pins" "1=D 2=G 3=S" (at 138.43 79.502 0)
+    (property "Sim.Pins" "1=D 2=G 3=S" (at 134.62 77.47 0)
       (effects (font (size 1.27 1.27)) hide)
     )
@@
     )
   )
-  (symbol (lib_id "Simulation_SPICE:NMOS") (at 113.538 64.008 0) (unit 1)
+  (symbol (lib_id "Simulation_SPICE:NMOS") (at 109.22 62.23 0) (unit 1)
     (in_bom yes) (on_board yes) (dnp no) (fields_autoplaced)
-    (property "Reference" "Q1" (at 119.38 62.738 0)
+    (property "Reference" "Q1" (at 115.062 60.96 0)
       (effects (font (size 1.27 1.27)) (justify left))
     )
-    (property "Value" "NMOS" (at 119.38 65.278 0)
+    (property "Value" "NMOS" (at 115.062 63.5 0)
       (effects (font (size 1.27 1.27)) (justify left))
     )
-    (property "Footprint" "" (at 118.618 61.468 0)
+    (property "Footprint" "" (at 114.3 59.69 0)
       (effects (font (size 1.27 1.27)) hide)
     )
-    (property "Datasheet" "https://ngspice.sourceforge.io/docs/ngspice-manual.pdf" (at 113.538 76.708 0)
+    (property "Datasheet" "https://ngspice.sourceforge.io/docs/ngspice-manual.pdf" (at 109.22 74.93 0)
       (effects (font (size 1.27 1.27)) hide)
     )
-    (property "Sim.Device" "NMOS" (at 113.538 81.153 0)
+    (property "Sim.Device" "NMOS" (at 109.22 79.375 0)
       (effects (font (size 1.27 1.27)) hide)
     )
-    (property "Sim.Type" "VDMOS" (at 113.538 83.058 0)
+    (property "Sim.Type" "VDMOS" (at 109.22 81.28 0)
       (effects (font (size 1.27 1.27)) hide)
     )
-    (property "Sim.Pins" "1=D 2=G 3=S" (at 113.538 79.248 0)
+    (property "Sim.Pins" "1=D 2=G 3=S" (at 109.22 77.47 0)
       (effects (font (size 1.27 1.27)) hide)
     )
@@
     )
   )
-  (symbol (lib_id "Simulation_SPICE:NMOS") (at 113.792 78.74 0) (unit 1)
+  (symbol (lib_id "Simulation_SPICE:NMOS") (at 109.22 77.47 0) (unit 1)
     (in_bom yes) (on_board yes) (dnp no) (fields_autoplaced)
-    (property "Reference" "Q2" (at 119.634 77.47 0)
+    (property "Reference" "Q2" (at 115.062 76.2 0)
       (effects (font (size 1.27 1.27)) (justify left))
     )
-    (property "Value" "NMOS" (at 119.634 80.01 0)
+    (property "Value" "NMOS" (at 115.062 78.74 0)
       (effects (font (size 1.27 1.27)) (justify left))
     )
-    (property "Footprint" "" (at 118.872 76.2 0)
+    (property "Footprint" "" (at 114.3 74.93 0)
       (effects (font (size 1.27 1.27)) hide)
     )
-    (property "Datasheet" "https://ngspice.sourceforge.io/docs/ngspice-manual.pdf" (at 113.792 91.44 0)
+    (property "Datasheet" "https://ngspice.sourceforge.io/docs/ngspice-manual.pdf" (at 109.22 90.17 0)
       (effects (font (size 1.27 1.27)) hide)
     )
-    (property "Sim.Device" "NMOS" (at 113.792 95.885 0)
+    (property "Sim.Device" "NMOS" (at 109.22 94.615 0)
       (effects (font (size 1.27 1.27)) hide)
     )
-    (property "Sim.Type" "VDMOS" (at 113.792 97.79 0)
+    (property "Sim.Type" "VDMOS" (at 109.22 96.52 0)
       (effects (font (size 1.27 1.27)) hide)
     )
-    (property "Sim.Pins" "1=D 2=G 3=S" (at 113.792 93.98 0)
+    (property "Sim.Pins" "1=D 2=G 3=S" (at 109.22 92.71 0)
       (effects (font (size 1.27 1.27)) hide)
     )
